Commit message: added navigation launch file

File: src/mapper_description/urdf/mobile_base.xacro (robot description, xacro)
@@ -48,5 +48,5 @@
         <visual>
             <geometry>
-                <sphere radius="0.0315" />
+                <sphere radius="0.031" />
             </geometry>
             <origin xyz="0 0 0" rpy="0 0 0" />
@@ -55,5 +55,5 @@
         <collision>
             <geometry>
-                <sphere radius="0.0315" />
+                <sphere radius="0.031" />
             </geometry>
             <origin xyz="0 0 0" rpy="0 0 0" />
@@ -68,5 +68,5 @@
         <visual>
             <geometry>
-                <sphere radius="0.0315" />
+                <sphere radius="0.031" />
             </geometry>
             <origin xyz="0 0 0" rpy="0 0 0" />
@@ -75,5 +75,5 @@
         <collision>
             <geometry>
-                <sphere radius="0.0315" />
+                <sphere radius="0.031" />
             </geometry>
             <origin xyz="0 0 0" rpy="0 0 0" />
@@ -88,5 +88,5 @@
         <visual>
             <geometry>
-                <sphere radius="0.0315" />
+                <sphere radius="0.031" />
             </geometry>
             <origin xyz="0 0 0" rpy="0 0 0" />
@@ -95,5 +95,5 @@
         <collision>
             <geometry>
-                <sphere radius="0.0315" />
+                <sphere radius="0.031" />
             </geometry>
             <origin xyz="0 0 0" rpy="0 0 0" />
@@ -108,5 +108,5 @@
         <visual>
             <geometry>
-                <sphere radius="0.0315" />
+                <sphere radius="0.031" />
             </geometry>
             <origin xyz="0 0 0" rpy="0 0 0" />
@@ -115,5 +115,5 @@
         <collision>
             <geometry>
-                <sphere radius="0.0315" />
+                <sphere radius="0.031  " />
             </geometry>
             <origin xyz="0 0 0" rpy="0 0 0" />
