Commit message: updated the simulation world

File: install/mapper_description/share/mapper_description/urdf/common_properties.xacro (robot description, xacro)
@@ -1,36 +1 @@
-<?xml version="1.0"?>
-<robot xmlns:xacro="http://www.ros.org/wiki/xacro">
-    <material name="blue">
-        <color rgba="0 0 0.5 1" />
-    </material>
-    <material name="grey">
-        <color rgba="0.5 0.5 0.5 1" />
-    </material>
-    <xacro:macro name="box_inertia" params="m l w h xyz rpy">
-        <inertial>
-            <origin xyz="${xyz}" rpy="${rpy}" />
-            <mass value="${m}" />
-            <inertia ixx="${(m/12) * (h*h + l*l)}" ixy="0" ixz="0"
-                     iyy="${(m/12) * (w*w + l*l)}" iyz="0"
-                     izz="${(m/12) * (w*w + h*h)}" />
-        </inertial>
-    </xacro:macro>
-    <xacro:macro name="cylinder_inertia" params="m r h xyz rpy">
-        <inertial>
-            <origin xyz="${xyz}" rpy="${rpy}" />
-            <mass value="${m}" />
-            <inertia ixx="${(m/12) * (3*r*r + h*h)}" ixy="0" ixz="0"
-                     iyy="${(m/12) * (3*r*r + h*h)}" iyz="0"
-                     izz="${(m/2) * (r*r)}" />
-        </inertial>
-    </xacro:macro>
-    <xacro:macro name="sphere_inertia" params="m r xyz rpy">
-        <inertial>
-            <origin xyz="${xyz}" rpy="${rpy}" />
-            <mass value="${m}" />
-            <inertia ixx="${(2/5) * m * r * r}" ixy="0" ixz="0"
-                     iyy="${(2/5) * m * r * r}" iyz="0"
-                     izz="${(2/5) * m * r * r}" />
-        </inertial>
-    </xacro:macro>
-</robot>
+/home/pranav/the_mapper/src/mapper_description/urdf/common_properties.xacro

File: install/mapper_description/share/mapper_description/urdf/mapper.urdf.xacro (robot description, xacro)
@@ -1,7 +1 @@
-<?xml version="1.0"?>
-<robot name="mapper" xmlns:xacro="http://www.ros.org/wiki/xacro">
-    <xacro:include filename="common_properties.xacro" />
-    <xacro:include filename="mobile_base.xacro" />
-    <xacro:include filename="mobile_base_gazebo.xacro" />
-    <xacro:include filename="sensors.xacro" />
-</robot>
+/home/pranav/the_mapper/src/mapper_description/urdf/mapper.urdf.xacro

File: install/mapper_description/share/mapper_description/urdf/mobile_base.xacro (robot description, xacro)
@@ -1,164 +1 @@
-<?xml version="1.0"?>
-<robot xmlns:xacro="http://www.ros.org/wiki/xacro">
-    <xacro:property name="base_length" value="0.65" />
-    <xacro:property name="base_width" value="0.45" />
-    <xacro:property name="base_height" value="0.2" />
-    <xacro:property name="wheel_radius" value="0.063" />
-    <xacro:property name="wheel_length" value="0.05" />
-    <link name="base_footprint" />
-    <link name="base_link">
-        <visual>
-            <geometry>
-                <box size="${base_length} ${base_width} ${base_height}" />
-            </geometry>
-            <origin xyz="0 0 ${base_height / 2.0}" rpy="0 0 0" />
-            <material name="blue" />
-        </visual>
-        <collision>
-            <geometry>
-                <box size="${base_length} ${base_width} ${base_height}" />
-            </geometry>
-            <origin xyz="0 0 ${base_height / 2.0}" rpy="0 0 0" />
-        </collision>
-        <xacro:box_inertia m="5.0" l="${2*base_length}" w="${2*base_width}" h="${2*base_height}"
-                           xyz="0 0 ${base_height / 2.0}" rpy="0 0 0" />
-    </link>
-    <xacro:macro name="wheel_link" params="prefix">
-        <link name="${prefix}_wheel_link">
-            <visual>
-                <geometry>
-                    <cylinder radius="${wheel_radius}" length="${wheel_length}" />
-                </geometry>
-                <origin xyz="0 0 0" rpy="${pi / 2.0} 0 0" />
-                <material name="grey" />
-            </visual>
-            <collision>
-                <geometry>
-                    <cylinder radius="${wheel_radius}" length="${wheel_length}" />
-                </geometry>
-                <origin xyz="0 0 0" rpy="${pi / 2.0} 0 0" />
-            </collision>
-            <xacro:cylinder_inertia m="1.0" r="${2*wheel_radius}" h="${2*wheel_length}"
-                                    xyz="0 0 0" rpy="${pi / 2.0} 0 0" />
-        </link>
-    </xacro:macro>
-    <xacro:wheel_link prefix="right" />
-    <xacro:wheel_link prefix="left" />
-   <link name="caster_wheel_link_1">
-        <visual>
-            <geometry>
-                <sphere radius="0.0315" />
-            </geometry>
-            <origin xyz="0 0 0" rpy="0 0 0" />
-            <material name="grey" />
-        </visual>
-        <collision>
-            <geometry>
-                <sphere radius="0.0315" />
-            </geometry>
-            <origin xyz="0 0 0" rpy="0 0 0" />
-        </collision>
-        <inertial>
-            <origin xyz="0 0 0" rpy="0 0 0" />
-            <mass value="0.2" />
-            <inertia ixx="0.00007938" ixy="0.0" ixz="0.0" iyy="0.00007938" iyz="0.0" izz="0.00007938" />
-        </inertial>
-    </link>
-    <link name="caster_wheel_link_2">
-        <visual>
-            <geometry>
-                <sphere radius="0.0315" />
-            </geometry>
-            <origin xyz="0 0 0" rpy="0 0 0" />
-            <material name="grey" />
-        </visual>
-        <collision>
-            <geometry>
-                <sphere radius="0.0315" />
-            </geometry>
-            <origin xyz="0 0 0" rpy="0 0 0" />
-        </collision>
-        <inertial>
-            <origin xyz="0 0 0" rpy="0 0 0" />
-            <mass value="0.2" />
-            <inertia ixx="0.00007938" ixy="0.0" ixz="0.0" iyy="0.00007938" iyz="0.0" izz="0.00007938" />
-        </inertial>
-    </link>
-    <link name="caster_wheel_link_3">
-        <visual>
-            <geometry>
-                <sphere radius="0.0315" />
-            </geometry>
-            <origin xyz="0 0 0" rpy="0 0 0" />
-            <material name="grey" />
-        </visual>
-        <collision>
-            <geometry>
-                <sphere radius="0.0315" />
-            </geometry>
-            <origin xyz="0 0 0" rpy="0 0 0" />
-        </collision>
-        <inertial>
-            <origin xyz="0 0 0" rpy="0 0 0" />
-            <mass value="0.2" />
-            <inertia ixx="0.00007938" ixy="0.0" ixz="0.0" iyy="0.00007938" iyz="0.0" izz="0.00007938" />
-        </inertial>
-    </link>
-    <link name="caster_wheel_link_4">
-        <visual>
-            <geometry>
-                <sphere radius="0.0315" />
-            </geometry>
-            <origin xyz="0 0 0" rpy="0 0 0" />
-            <material name="grey" />
-        </visual>
-        <collision>
-            <geometry>
-                <sphere radius="0.0315" />
-            </geometry>
-            <origin xyz="0 0 0" rpy="0 0 0" />
-        </collision>
-        <inertial>
-            <origin xyz="0 0 0" rpy="0 0 0" />
-            <mass value="0.2" />
-            <inertia ixx="0.00007938" ixy="0.0" ixz="0.0" iyy="0.00007938" iyz="0.0" izz="0.00007938" />
-        </inertial>
-    </link>
-    <joint name="base_joint" type="fixed">
-        <parent link="base_footprint" />
-        <child link="base_link" />
-        <origin xyz="0 0 ${wheel_radius}" rpy="0 0 0"/>
-    </joint>
-    <joint name="base_right_wheel_joint" type="continuous">
-        <parent link="base_link" />
-        <child link="right_wheel_link" />
-        <origin xyz="0 -0.225 0" rpy="0 0 0" />
-        <axis xyz="0 1 0" />
-    </joint>
-    <joint name="base_left_wheel_joint" type="continuous">
-        <parent link="base_link" />
-        <child link="left_wheel_link" />
-        <origin xyz="0 0.225 0" rpy="0 0 0" />
-        <axis xyz="0 1 0" />
-    </joint>
-    <joint name="base_caster_wheel_1_joint" type="fixed">
-        <parent link="base_link" />
-        <child link="caster_wheel_link_1" />
-        <origin xyz="-0.181 -0.15 -0.0315" rpy="0 0 0" />
-    </joint>
-    <joint name="base_caster_wheel_2_joint" type="fixed">
-        <parent link="base_link" />
-        <child link="caster_wheel_link_2" />
-        <origin xyz="-0.181 0.15 -0.0315" rpy="0 0 0" />
-    </joint>
-    <joint name="base_caster_wheel_3_joint" type="fixed">
-        <parent link="base_link" />
-        <child link="caster_wheel_link_3" />
-        <origin xyz="0.181 0.15 -0.0315" rpy="0 0 0" />
-    </joint>
-    <joint name="base_caster_wheel_4_joint" type="fixed">
-        <parent link="base_link" />
-        <child link="caster_wheel_link_4" />
-        <origin xyz="0.181 -0.15 -0.0315" rpy="0 0 0" />
-    </joint>
-</robot>
+/home/pranav/the_mapper/src/mapper_description/urdf/mobile_base.xacro

File: install/mapper_description/share/mapper_description/urdf/mobile_base_gazebo.xacro (robot description, xacro)
@@ -1,78 +1 @@
-<?xml version="1.0"?>
-<robot xmlns:xacro="http://www.ros.org/wiki/xacro">
-    <gazebo reference="base_link">
-        <material>Gazebo/Blue</material>
-    </gazebo>
-    <gazebo reference="right_wheel_link">
-        <material>Gazebo/Grey</material>
-    </gazebo>
-    <gazebo reference="left_wheel_link">
-        <material>Gazebo/Grey</material>
-    </gazebo>
-    <gazebo reference="caster_wheel_link_1">
-        <material>Gazebo/Grey</material>
-        <mu1 value="0.1" />
-        <mu2 value="0.1" />
-    </gazebo>
-    <gazebo reference="caster_wheel_link_2">
-        <material>Gazebo/Grey</material>
-        <mu1 value="0.1" />
-        <mu2 value="0.1" />
-    </gazebo>
-    <gazebo reference="caster_wheel_link_3">
-        <material>Gazebo/Grey</material>
-        <mu1 value="0.1" />
-        <mu2 value="0.1" />
-    </gazebo>
-    <gazebo reference="caster_wheel_link_4">
-        <material>Gazebo/Grey</material>
-        <mu1 value="0.1" />
-        <mu2 value="0.1" />
-    </gazebo>
-    <gazebo reference="lidar_link">
-        <material>Gazebo/Grey</material>
-        <mu1 value="0.1" />
-        <mu2 value="0.1" />
-    </gazebo>
-    <gazebo>
-        <plugin name="diff_drive_controller" filename="libgazebo_ros_diff_drive.so">
-            <!-- Update rate in Hz -->
-            <update_rate>50</update_rate>
-            <!-- wheels -->
-            <left_joint>base_left_wheel_joint</left_joint>
-            <right_joint>base_right_wheel_joint</right_joint>
-            <!-- kinematics -->
-            <wheel_separation>0.39</wheel_separation>
-            <wheel_diameter>0.127</wheel_diameter>
-            <!-- output -->
-            <publish_odom>true</publish_odom>
-            <publish_odom_tf>true</publish_odom_tf>
-            <publish_wheel_tf>true</publish_wheel_tf>
-            <odometry_topic>odom</odometry_topic>
-            <odometry_frame>odom</odometry_frame>
-            <robot_base_frame>base_footprint</robot_base_frame>
-            <max_speed>10.0</max_speed>
-            <max_turning_speed>2.0</max_turning_speed>
-        </plugin>
-    </gazebo>
-    <gazebo reference="imu_link">
-        <gravity>true</gravity>
-        <sensor name="imu_sensor" type="imu">
-            <always_on>true</always_on>
-            <update_rate>50</update_rate>
-            <visualize>true</visualize>
-            <topic>imu1</topic>
-            <plugin name="imu_plugin" filename="libgazebo_ros_imu_sensor.so">
-                <topicName>imu</topicName>
-                <bodyName>imu_link</bodyName>
-                <updateRateHZ>10.0</updateRateHZ>
-                <gaussianNoise>0.0</gaussianNoise>
-                <xyzOffset>0 0 0</xyzOffset>
-                <rpyOffset>0 0 0</rpyOffset>
-                <frameName>imu_link</frameName>
-                <initialOrientationAsReference>false</initialOrientationAsReference>
-            </plugin>
-            <pose>0 0 0 0 0 0</pose>
-        </sensor>
-  </gazebo>
-</robot>
+/home/pranav/the_mapper/src/mapper_description/urdf/mobile_base_gazebo.xacro

File: install/mapper_description/share/mapper_description/urdf/sensors.xacro (robot description, xacro)
@@ -1,71 +1 @@
-<?xml version="1.0"?>
-<robot xmlns:xacro="http://www.ros.org/wiki/xacro" >
-    <joint name="lidar_joint" type="fixed">
-        <parent link="base_link"/>
-        <child link="lidar_link"/>
-        <origin xyz="0 0 0.21" rpy="0 0 0"/>
-    </joint>
-    <link name="lidar_link">
-        <visual>
-            <geometry>
-                <cylinder radius="0.05" length="0.05"/>
-            </geometry>
-            <material name="grey"/>
-        </visual>
-        <collision>
-            <geometry>
-                <cylinder radius="0.05" length="0.05"/>
-            </geometry>
-        </collision>
-        <xacro:box_inertia m="5.0" l="${2*base_length}" w="${2*base_width}" h="${2*base_height}"
-                           xyz="0 0 ${base_height / 2.0}" rpy="0 0 0" />
-    </link>
-    <joint name="imu_joint" type="fixed">
-        <parent link="base_link"/>
-        <child link="imu_link"/>
-        <origin xyz="0 0 0.1" rpy="0 0 0"/>
-    </joint>
-    <link name="imu_link">
-        <visual>
-            <geometry>
-                <box size="0.05 0.05 0.02"/>
-            </geometry>
-            <material name="grey"/>
-        </visual>
-        <collision>
-            <geometry>
-                <box size="0.1 0.1 0.1"/>
-            </geometry>
-        </collision>
-        <xacro:box_inertia m="0.1" l="0.1" w="0.1" h="0.1"
-                           xyz="0 0 0" rpy="0 0 0" />
-    </link>
-    <gazebo reference="lidar_link">
-        <material>Gazebo/Grey</material>
-        <sensor name="laser" type="ray">
-            <pose> 0 0 0 0 0 0 </pose>
-            <visualize>true</visualize>
-            <update_rate>10</update_rate>
-            <ray>
-                <scan>
-                    <horizontal>
-                        <samples>360</samples>
-                        <min_angle>-3.14</min_angle>
-                        <max_angle>3.14</max_angle>
-                    </horizontal>
-                </scan>
-                <range>
-                    <min>0.3</min>
-                    <max>12</max>
-                </range>
-            </ray>
-            <plugin name="laser_controller" filename="libgazebo_ros_ray_sensor.so">
-                <ros>
-                    <argument>~/out:=scan</argument>
-                </ros>
-                <output_type>sensor_msgs/LaserScan</output_type>
-                <frame_name>lidar_link</frame_name>
-            </plugin>
-        </sensor>
-    </gazebo>
-</robot>
+/home/pranav/the_mapper/src/mapper_description/urdf/sensors.xacro

File: src/mapper_description/urdf/mobile_base.xacro (robot description, xacro)
@@ -48,5 +48,5 @@
         <visual>
             <geometry>
-                <sphere radius="0.031" />
+                <sphere radius="0.0315" />
             </geometry>
             <origin xyz="0 0 0" rpy="0 0 0" />
@@ -55,5 +55,5 @@
         <collision>
             <geometry>
-                <sphere radius="0.031" />
+                <sphere radius="0.0315" />
             </geometry>
             <origin xyz="0 0 0" rpy="0 0 0" />
@@ -68,5 +68,5 @@
         <visual>
             <geometry>
-                <sphere radius="0.031" />
+                <sphere radius="0.0315" />
             </geometry>
             <origin xyz="0 0 0" rpy="0 0 0" />
@@ -75,5 +75,5 @@
         <collision>
             <geometry>
-                <sphere radius="0.031" />
+                <sphere radius="0.0315" />
             </geometry>
             <origin xyz="0 0 0" rpy="0 0 0" />
@@ -88,5 +88,5 @@
         <visual>
             <geometry>
-                <sphere radius="0.031" />
+                <sphere radius="0.0315" />
             </geometry>
             <origin xyz="0 0 0" rpy="0 0 0" />
@@ -95,5 +95,5 @@
         <collision>
             <geometry>
-                <sphere radius="0.031" />
+                <sphere radius="0.0315" />
             </geometry>
             <origin xyz="0 0 0" rpy="0 0 0" />
@@ -108,5 +108,5 @@
         <visual>
             <geometry>
-                <sphere radius="0.031" />
+                <sphere radius="0.0315" />
             </geometry>
             <origin xyz="0 0 0" rpy="0 0 0" />
@@ -115,5 +115,5 @@
         <collision>
             <geometry>
-                <sphere radius="0.031  " />
+                <sphere radius="0.0315" />
             </geometry>
             <origin xyz="0 0 0" rpy="0 0 0" />
