Commit message: Update

File: install/mapper_description/share/mapper_description/urdf/mobile_base_gazebo.xacro (robot description, xacro)
@@ -6,21 +6,21 @@
     <gazebo reference="right_wheel_link">
         <material>Gazebo/Grey</material>
-        <mu1 value="0.3" />
-        <mu2 value="0.3" />
+        <mu1 value="100" />
+        <mu2 value="100" />
     </gazebo>
     <gazebo reference="left_wheel_link">
         <material>Gazebo/Grey</material>
-        <mu1 value="0.3" />
-        <mu2 value="0.3" />
+        <mu1 value="100" />
+        <mu2 value="100" />
     </gazebo>
     <gazebo reference="rightb_wheel_link">
         <material>Gazebo/Grey</material>
-        <mu1 value="0.3" />
-        <mu2 value="0.3" />
+        <mu1 value="100" />
+        <mu2 value="100" />
     </gazebo>
     <gazebo reference="leftb_wheel_link">
         <material>Gazebo/Grey</material>
-        <mu1 value="0.3" />
-        <mu2 value="0.3" />
+        <mu1 value="100" />
+        <mu2 value="100" />
     </gazebo>
     <gazebo reference="lidar_link">

File: install/mapper_description/share/mapper_description/urdf/sensors.xacro (robot description, xacro)
@@ -1,4 +1,29 @@
 <?xml version="1.0"?>
 <robot xmlns:xacro="http://www.ros.org/wiki/xacro" >
+    <joint name="sonar_front_joint" type="fixed">
+        <axis xyz="0 1 0" />
+        <origin rpy="0 0 0" xyz="0.16 0 0.09" />
+        <parent link="base_footprint"/>
+        <child link="base_sonar_front"/>
+    </joint>
+    <link name="base_sonar_front">
+        <collision>
+          <origin xyz="0 0 0" rpy="0 0 0"/>
+          <geometry>
+            <box size="0.01 0.01 0.01"/>
+          </geometry>
+        </collision>
+        <visual>
+          <origin xyz="0 0 0" rpy="0 0 0"/>
+          <geometry>
+            <box size="0.01 0.01 0.01"/>
+          </geometry>
+        </visual>
+        <inertial>
+          <mass value="1e-5" />
+          <origin xyz="0 0 0" rpy="0 0 0"/>
+          <inertia ixx="1e-6" ixy="0" ixz="0" iyy="1e-6" iyz="0" izz="1e-6" />
+        </inertial>
+     </link>
     <joint name="lidar_joint" type="fixed">
         <parent link="base_footprint"/>
@@ -69,3 +94,42 @@
         </sensor>
     </gazebo>
+    <gazebo reference="base_sonar_front">
+        <sensor type="ray" name="TeraRanger">
+            <pose>0 0 0 0 0 0</pose>
+            <visualize>true</visualize>
+            <update_rate>50</update_rate>
+            <ray>
+                <scan>
+                    <horizontal>
+                        <samples>10</samples>
+                        <resolution>1</resolution>
+                        <min_angle>-0.18326</min_angle>
+                        <max_angle>0.18326</max_angle>
+                    </horizontal>
+                    <vertical>
+                        <samples>1</samples>
+                        <resolution>1</resolution>
+                        <min_angle>0</min_angle>
+                        <max_angle>0</max_angle>
+                    </vertical>
+                </scan>
+                <range>
+                    <min>0.01</min>
+                    <max>2</max>
+                    <resolution>0.02</resolution>
+                </range>
+            </ray>
+            <plugin name="gazebo_ros_range_sensor" filename="libgazebo_ros_ray_sensor.so">
+                <ros>
+                    <namespace>sensor</namespace>
+                    <argument>sonar_front:=sonar_front</argument>
+                </ros>
+                <topicName>/sensor/sonar_front</topicName>
+                <frameName>base_sonar_front</frameName>
+                <updateRate>50</updateRate>
+                <gaussianNoise>0.005</gaussianNoise>
+                <radiation>INFRARED</radiation>
+            </plugin>
+        </sensor>
+    </gazebo>
 </robot>

File: src/mapper_description/urdf/mobile_base_gazebo.xacro (robot description, xacro)
@@ -6,21 +6,21 @@
     <gazebo reference="right_wheel_link">
         <material>Gazebo/Grey</material>
-        <mu1 value="0.3" />
-        <mu2 value="0.3" />
+        <mu1 value="1" />
+        <mu2 value="1" />
     </gazebo>
     <gazebo reference="left_wheel_link">
         <material>Gazebo/Grey</material>
-        <mu1 value="0.3" />
-        <mu2 value="0.3" />
+        <mu1 value="1" />
+        <mu2 value="1" />
     </gazebo>
     <gazebo reference="rightb_wheel_link">
         <material>Gazebo/Grey</material>
-        <mu1 value="0.3" />
-        <mu2 value="0.3" />
+        <mu1 value="1" />
+        <mu2 value="0.5" />
     </gazebo>
     <gazebo reference="leftb_wheel_link">
         <material>Gazebo/Grey</material>
-        <mu1 value="0.3" />
-        <mu2 value="0.3" />
+        <mu1 value="0.5" />
+        <mu2 value="0.5" />
     </gazebo>
     <gazebo reference="lidar_link">

Commit message: Reworking sensor fusion

File: install/mapper_description/share/mapper_description/urdf/mobile_base_gazebo.xacro (robot description, xacro)
@@ -8,4 +8,7 @@
         <mu1 value="0.7" />
         <mu2 value="0.5" />
+    </gazebo>
+    <gazebo reference="base_sonar_front">
+        <material>Gazebo/Grey</material>
     </gazebo>
     <gazebo reference="left_wheel_link">

File: install/mapper_description/share/mapper_description/urdf/sensors.xacro (robot description, xacro)
@@ -19,4 +19,5 @@
             <box size="0.01 0.01 0.01"/>
           </geometry>
+          <material name="grey"/>
         </visual>
         <inertial>
