Commit message: u3

File: install/mapper_description/share/mapper_description/urdf/mobile_base.xacro (robot description, xacro)
@@ -5,5 +5,5 @@
     <xacro:property name="base_height" value="0.08" />
     <xacro:property name="wheel_radius" value="0.05" />
-    <xacro:property name="wheel_length" value="0.05" />
+    <xacro:property name="wheel_length" value="0.03" />
     <link name="base_footprint" />
     <link name="base_link">

File: install/mapper_description/share/mapper_description/urdf/mobile_base_gazebo.xacro (robot description, xacro)
@@ -6,6 +6,6 @@
     <gazebo reference="right_wheel_link">
         <material>Gazebo/Grey</material>
-        <mu1 value="0.7" />
-        <mu2 value="0.5" />
+        <mu1 value="0.5" />
+        <mu2 value="0.4" />
     </gazebo>
     <gazebo reference="base_sonar_front">
@@ -14,16 +14,16 @@
     <gazebo reference="left_wheel_link">
         <material>Gazebo/Grey</material>
-        <mu1 value="0.7" />
-        <mu2 value="0.5" />
+        <mu1 value="0.5" />
+        <mu2 value="0.4" />
     </gazebo>
     <gazebo reference="rightb_wheel_link">
         <material>Gazebo/Grey</material>
-        <mu1 value="0.7" />
-        <mu2 value="0.5" />
+        <mu1 value="0.5" />
+        <mu2 value="0.4" />
     </gazebo>
     <gazebo reference="leftb_wheel_link">
         <material>Gazebo/Grey</material>
-        <mu1 value="0.7" />
-        <mu2 value="0.5" />
+        <mu1 value="0.5" />
+        <mu2 value="0.4" />
     </gazebo>
     <gazebo reference="lidar_link">
@@ -32,5 +32,5 @@
     <gazebo>
         <plugin name="skid_steer_drive_controller" filename="libgazebo_ros_diff_drive.so">
-            <update_rate>50</update_rate>
+            <update_rate>100</update_rate>
             <num_wheel_pairs>2</num_wheel_pairs>
             <left_joint>base_leftb_wheel_joint</left_joint>
@@ -38,8 +38,8 @@
             <left_joint>base_left_wheel_joint</left_joint>
             <right_joint>base_right_wheel_joint</right_joint>
-            <wheel_separation>0.015</wheel_separation>
+            <wheel_separation>0.18</wheel_separation>
             <wheel_diameter>0.05</wheel_diameter>
             <max_wheel_torque>20</max_wheel_torque>
-            <max_wheel_accleration>3.0</max_wheel_accleration>
+            <max_wheel_acceleration>1.0</max_wheel_acceleration>
             <publish_odom>true</publish_odom>
             <publish_odom_tf>true</publish_odom_tf>

File: install/mapper_description/share/mapper_description/urdf/sensors.xacro (robot description, xacro)
@@ -72,5 +72,5 @@
             <pose> 0 0 0 0 0 0 </pose>
             <visualize>true</visualize>
-            <update_rate>10</update_rate>
+            <update_rate>100</update_rate>
             <ray>
                 <scan>
