Commit message: huge leap

File: install/mapper_description/share/mapper_description/urdf/mapper.urdf.xacro (robot description, xacro)
@@ -1,7 +1 @@
-<?xml version="1.0"?>
-<robot name="mapper" xmlns:xacro="http://www.ros.org/wiki/xacro">
-    <xacro:include filename="common_properties.xacro" />
-    <xacro:include filename="mobile_base.xacro" />
-    <xacro:include filename="mobile_base_gazebo.xacro" />
-    <xacro:include filename="sensors.xacro" />
-</robot>
+/home/pranav/the_mapper/src/mapper_description/urdf/mapper.urdf.xacro

File: install/mapper_description/share/mapper_description/urdf/mobile_base.xacro (robot description, xacro)
@@ -1,178 +1 @@
-<?xml version="1.0"?>
-<robot xmlns:xacro="http://www.ros.org/wiki/xacro">
-    <xacro:property name="base_length" value="0.30" />
-    <xacro:property name="base_width" value="0.15" />
-    <xacro:property name="base_height" value="0.08" />
-    <xacro:property name="wheel_radius" value="0.05" />
-    <xacro:property name="wheel_length" value="0.03" />
-    <link name="base_footprint" />
-    <link name="base_link">
-        <visual>
-            <geometry>
-                <box size="${base_length} ${base_width} ${base_height}" />
-            </geometry>
-            <origin xyz="0 0 ${base_height / 2.0}" rpy="0 0 0" />
-            <material name="blue" />
-        </visual>
-        <collision>
-            <geometry>
-                <box size="${base_length} ${base_width} ${base_height}" />
-            </geometry>
-            <origin xyz="0 0 ${base_height / 2.0}" rpy="0 0 0" />
-        </collision>
-        <xacro:box_inertia m="5.0" l="${2*base_length}" w="${2*base_width}" h="${2*base_height}"
-                           xyz="0 0 ${base_height / 2.0}" rpy="0 0 0" />
-    </link>
-    <xacro:macro name="wheel_link" params="prefix">
-        <link name="${prefix}_wheel_link">
-            <visual>
-                <geometry>
-                    <cylinder radius="${wheel_radius}" length="${wheel_length}" />
-                </geometry>
-                <origin xyz="0 0 0" rpy="${pi / 2.0} 0 0" />
-                <material name="grey" />
-            </visual>
-            <collision>
-                <geometry>
-                    <cylinder radius="${wheel_radius}" length="${wheel_length}" />
-                </geometry>
-                <origin xyz="0 0 0" rpy="${pi / 2.0} 0 0" />
-            </collision>
-            <xacro:cylinder_inertia m="1.0" r="${2*wheel_radius}" h="${2*wheel_length}"
-                                    xyz="0 0 0" rpy="${pi / 2.0} 0 0" />
-        </link>
-    </xacro:macro>
-    <xacro:wheel_link prefix="right" />
-    <xacro:wheel_link prefix="left" />
-    <xacro:wheel_link prefix="rightb" />
-    <xacro:wheel_link prefix="leftb" />
-   <!-- <link name="caster_wheel_link_1">
-        <visual>
-            <geometry>
-                <sphere radius="0.0315" />
-            </geometry>
-            <origin xyz="0 0 0" rpy="0 0 0" />
-            <material name="grey" />
-        </visual>
-        <collision>
-            <geometry>
-                <sphere radius="0.0315" />
-            </geometry>
-            <origin xyz="0 0 0" rpy="0 0 0" />
-        </collision>
-        <inertial>
-            <origin xyz="0 0 0" rpy="0 0 0" />
-            <mass value="0.2" />
-            <inertia ixx="0.00007938" ixy="0.0" ixz="0.0" iyy="0.00007938" iyz="0.0" izz="0.00007938" />
-        </inertial>
-    </link>
-    <link name="caster_wheel_link_2">
-        <visual>
-            <geometry>
-                <sphere radius="0.0315" />
-            </geometry>
-            <origin xyz="0 0 0" rpy="0 0 0" />
-            <material name="grey" />
-        </visual>
-        <collision>
-            <geometry>
-                <sphere radius="0.0315" />
-            </geometry>
-            <origin xyz="0 0 0" rpy="0 0 0" />
-        </collision>
-        <inertial>
-            <origin xyz="0 0 0" rpy="0 0 0" />
-            <mass value="0.2" />
-            <inertia ixx="0.00007938" ixy="0.0" ixz="0.0" iyy="0.00007938" iyz="0.0" izz="0.00007938" />
-        </inertial>
-    </link>
-    <link name="caster_wheel_link_3">
-        <visual>
-            <geometry>
-                <sphere radius="0.0315" />
-            </geometry>
-            <origin xyz="0 0 0" rpy="0 0 0" />
-            <material name="grey" />
-        </visual>
-        <collision>
-            <geometry>
-                <sphere radius="0.0315" />
-            </geometry>
-            <origin xyz="0 0 0" rpy="0 0 0" />
-        </collision>
-        <inertial>
-            <origin xyz="0 0 0" rpy="0 0 0" />
-            <mass value="0.2" />
-            <inertia ixx="0.00007938" ixy="0.0" ixz="0.0" iyy="0.00007938" iyz="0.0" izz="0.00007938" />
-        </inertial>
-    </link>
-    <link name="caster_wheel_link_4">
-        <visual>
-            <geometry>
-                <sphere radius="0.0315" />
-            </geometry>
-            <origin xyz="0 0 0" rpy="0 0 0" />
-            <material name="grey" />
-        </visual>
-        <collision>
-            <geometry>
-                <sphere radius="0.0315" />
-            </geometry>
-            <origin xyz="0 0 0" rpy="0 0 0" />
-        </collision>
-        <inertial>
-            <origin xyz="0 0 0" rpy="0 0 0" />
-            <mass value="0.2" />
-            <inertia ixx="0.00007938" ixy="0.0" ixz="0.0" iyy="0.00007938" iyz="0.0" izz="0.00007938" />
-        </inertial>
-    </link> -->
-    <joint name="base_joint" type="fixed">
-        <parent link="base_footprint" />
-        <child link="base_link" />
-        <origin xyz="0 0 ${wheel_radius}" rpy="0 0 0"/>
-    </joint>
-    <joint name="base_right_wheel_joint" type="continuous">
-        <parent link="base_link" />
-        <child link="right_wheel_link" />
-        <origin xyz="0.09 -0.1 0" rpy="0 0 0" />
-        <axis xyz="0 1 0" />
-    </joint>
-    <joint name="base_left_wheel_joint" type="continuous">
-        <parent link="base_link" />
-        <child link="left_wheel_link" />
-        <origin xyz="0.09 0.1 0" rpy="0 0 0" />
-        <axis xyz="0 1 0" />
-    </joint>
-    <joint name="base_rightb_wheel_joint" type="continuous">
-        <parent link="base_link" />
-        <child link="rightb_wheel_link" />
-        <origin xyz="-0.09 -0.1 0" rpy="0 0 0" />
-        <axis xyz="0 1 0" />
-    </joint>
-    <joint name="base_leftb_wheel_joint" type="continuous">
-        <parent link="base_link" />
-        <child link="leftb_wheel_link" />
-        <origin xyz="-0.09 0.1 0" rpy="0 0 0" />
-        <axis xyz="0 1 0" />
-    </joint>
-    <!-- <joint name="base_caster_wheel_1_joint" type="fixed">
-        <parent link="base_link" />
-        <child link="caster_wheel_link_1" />
-        <origin xyz="-0.181 -0.15 -0.0315" rpy="0 0 0" />
-    </joint>
-    <joint name="base_caster_wheel_2_joint" type="fixed">
-        <parent link="base_link" />
-        <child link="caster_wheel_link_2" />
-        <origin xyz="-0.181 0.15 -0.0315" rpy="0 0 0" />
-    </joint>
-    <joint name="base_caster_wheel_3_joint" type="fixed">
-        <parent link="base_link" />
-        <child link="caster_wheel_link_3" />
-        <origin xyz="0.181 0.15 -0.0315" rpy="0 0 0" />
-    </joint>
-    <joint name="base_caster_wheel_4_joint" type="fixed">
-        <parent link="base_link" />
-        <child link="caster_wheel_link_4" />
-        <origin xyz="0.181 -0.15 -0.0315" rpy="0 0 0" />
-    </joint> -->
-</robot>
+/home/pranav/the_mapper/src/mapper_description/urdf/mobile_base.xacro

File: install/mapper_description/share/mapper_description/urdf/mobile_base_gazebo.xacro (robot description, xacro)
@@ -1,72 +1 @@
-<?xml version="1.0"?>
-<robot xmlns:xacro="http://www.ros.org/wiki/xacro">
-    <gazebo reference="base_link">
-        <material>Gazebo/Blue</material>
-    </gazebo>
-    <gazebo reference="right_wheel_link">
-        <material>Gazebo/Grey</material>
-        <mu1 value="0.5" />
-        <mu2 value="0.4" />
-    </gazebo>
-    <gazebo reference="base_sonar_front">
-        <material>Gazebo/Grey</material>
-    </gazebo>
-    <gazebo reference="left_wheel_link">
-        <material>Gazebo/Grey</material>
-        <mu1 value="0.5" />
-        <mu2 value="0.4" />
-    </gazebo>
-    <gazebo reference="rightb_wheel_link">
-        <material>Gazebo/Grey</material>
-        <mu1 value="0.5" />
-        <mu2 value="0.4" />
-    </gazebo>
-    <gazebo reference="leftb_wheel_link">
-        <material>Gazebo/Grey</material>
-        <mu1 value="0.5" />
-        <mu2 value="0.4" />
-    </gazebo>
-    <gazebo reference="lidar_link">
-        <material>Gazebo/Grey</material>
-    </gazebo>
-    <gazebo>
-        <plugin name="skid_steer_drive_controller" filename="libgazebo_ros_diff_drive.so">
-            <update_rate>50</update_rate>
-            <num_wheel_pairs>2</num_wheel_pairs>
-            <left_joint>base_leftb_wheel_joint</left_joint>
-            <right_joint>base_rightb_wheel_joint</right_joint>
-            <left_joint>base_left_wheel_joint</left_joint>
-            <right_joint>base_right_wheel_joint</right_joint>
-            <wheel_separation>0.18</wheel_separation>
-            <wheel_diameter>0.05</wheel_diameter>
-            <max_wheel_torque>20</max_wheel_torque>
-            <max_wheel_acceleration>1.0</max_wheel_acceleration>
-            <publish_odom>true</publish_odom>
-            <publish_odom_tf>true</publish_odom_tf>
-            <publish_wheel_tf>true</publish_wheel_tf>
-            <odometry_frame>odom</odometry_frame>
-            <odometry_topic>odom</odometry_topic>
-            <robot_base_frame>base_footprint</robot_base_frame>
-        </plugin>
-    </gazebo>
-    <gazebo reference="imu_link">
-        <gravity>true</gravity>
-        <sensor name="imu_sensor" type="imu">
-            <always_on>true</always_on>
-            <update_rate>50</update_rate>
-            <visualize>true</visualize>
-            <topic>imu1</topic>
-            <plugin name="imu_plugin" filename="libgazebo_ros_imu_sensor.so">
-                <topicName>imu1</topicName>
-                <bodyName>imu_link</bodyName>
-                <updateRateHZ>10.0</updateRateHZ>
-                <gaussianNoise>0.0</gaussianNoise>
-                <xyzOffset>0 0 0</xyzOffset>
-                <rpyOffset>0 0 0</rpyOffset>
-                <frameName>imu_link</frameName>
-                <initialOrientationAsReference>false</initialOrientationAsReference>
-            </plugin>
-            <pose>0 0 0 0 0 0</pose>
-        </sensor>
-  </gazebo>
-</robot>
+/home/pranav/the_mapper/src/mapper_description/urdf/mobile_base_gazebo.xacro

File: install/mapper_description/share/mapper_description/urdf/sensors.xacro (robot description, xacro)
@@ -1,136 +1 @@
-<?xml version="1.0"?>
-<robot xmlns:xacro="http://www.ros.org/wiki/xacro" >
-    <joint name="sonar_front_joint" type="fixed">
-        <axis xyz="0 1 0" />
-        <origin rpy="0 0 0" xyz="0.16 0 0.09" />
-        <parent link="base_footprint"/>
-        <child link="base_sonar_front"/>
-    </joint>
-    <link name="base_sonar_front">
-        <collision>
-          <origin xyz="0 0 0" rpy="0 0 0"/>
-          <geometry>
-            <box size="0.01 0.01 0.01"/>
-          </geometry>
-        </collision>
-        <visual>
-          <origin xyz="0 0 0" rpy="0 0 0"/>
-          <geometry>
-            <box size="0.01 0.01 0.01"/>
-          </geometry>
-          <material name="grey"/>
-        </visual>
-        <inertial>
-          <mass value="1e-5" />
-          <origin xyz="0 0 0" rpy="0 0 0"/>
-          <inertia ixx="1e-6" ixy="0" ixz="0" iyy="1e-6" iyz="0" izz="1e-6" />
-        </inertial>
-     </link>
-    <joint name="lidar_joint" type="fixed">
-        <parent link="base_footprint"/>
-        <child link="lidar_link"/>
-        <origin xyz="0 0 0.145" rpy="0 0 0"/>
-    </joint>
-    <link name="lidar_link">
-        <visual>
-            <geometry>
-                <cylinder radius="0.05" length="0.03"/>
-            </geometry>
-            <material name="grey"/>
-        </visual>
-        <collision>
-            <geometry>
-                <cylinder radius="0.05" length="0.03"/>
-            </geometry>
-        </collision>
-        <xacro:cylinder_inertia m="1.0" r="0.05" h="0.03"
-                                    xyz="0 0 0.095" rpy="0 0 0" />
-    </link>
-    <joint name="imu_joint" type="fixed">
-        <parent link="base_footprint"/>
-        <child link="imu_link"/>
-        <origin xyz="0 0 0.09" rpy="0 0 0"/>
-    </joint>
-    <link name="imu_link">
-        <visual>
-            <geometry>
-                <box size="0.05 0.05 0.02"/>
-            </geometry>
-            <material name="grey"/>
-        </visual>
-        <collision>
-            <geometry>
-                <box size="0.1 0.1 0.1"/>
-            </geometry>
-        </collision>
-        <xacro:box_inertia m="0.1" l="0.1" w="0.1" h="0.1"
-                           xyz="0 0 0" rpy="0 0 0" />
-    </link>
-    <gazebo reference="lidar_link">
-        <material>Gazebo/Grey</material>
-        <sensor name="laser" type="ray">
-            <pose> 0 0 0 0 0 0 </pose>
-            <visualize>true</visualize>
-            <update_rate>20</update_rate>
-            <ray>
-                <scan>
-                    <horizontal>
-                        <samples>360</samples>
-                        <min_angle>-3.14</min_angle>
-                        <max_angle>3.14</max_angle>
-                    </horizontal>
-                </scan>
-                <range>
-                    <min>0.3</min>
-                    <max>12</max>
-                </range>
-            </ray>
-            <plugin name="laser_controller" filename="libgazebo_ros_ray_sensor.so">
-                <ros>
-                    <argument>~/out:=scan</argument>
-                </ros>
-                <output_type>sensor_msgs/LaserScan</output_type>
-                <frame_name>lidar_link</frame_name>
-            </plugin>
-        </sensor>
-    </gazebo>
-    <gazebo reference="base_sonar_front">
-        <sensor type="ray" name="TeraRanger">
-            <pose>0 0 0 0 0 0</pose>
-            <visualize>true</visualize>
-            <update_rate>50</update_rate>
-            <ray>
-                <scan>
-                    <horizontal>
-                        <samples>10</samples>
-                        <resolution>1</resolution>
-                        <min_angle>-0.18326</min_angle>
-                        <max_angle>0.18326</max_angle>
-                    </horizontal>
-                    <vertical>
-                        <samples>1</samples>
-                        <resolution>1</resolution>
-                        <min_angle>0</min_angle>
-                        <max_angle>0</max_angle>
-                    </vertical>
-                </scan>
-                <range>
-                    <min>0.01</min>
-                    <max>2</max>
-                    <resolution>0.02</resolution>
-                </range>
-            </ray>
-            <plugin name="gazebo_ros_range_sensor" filename="libgazebo_ros_ray_sensor.so">
-                <ros>
-                    <namespace>sensor</namespace>
-                    <argument>sonar_front:=sonar_front</argument>
-                </ros>
-                <topicName>/sensor/sonar_front</topicName>
-                <frameName>base_sonar_front</frameName>
-                <updateRate>50</updateRate>
-                <gaussianNoise>0.005</gaussianNoise>
-                <radiation>INFRARED</radiation>
-            </plugin>
-        </sensor>
-    </gazebo>
-</robot>
+/home/pranav/the_mapper/src/mapper_description/urdf/sensors.xacro

File: src/mapper_description/urdf/mobile_base.xacro (robot description, xacro)
@@ -7,4 +7,9 @@
     <xacro:property name="wheel_length" value="0.03" />
     <link name="base_footprint" />
+    <joint name="base_joint" type="fixed">
+        <parent link="base_footprint" />
+        <child link="base_link" />
+        <origin xyz="0 0 ${wheel_radius}" rpy="0 0 0"/>
+    </joint>
     <link name="base_link">
         <visual>
@@ -127,13 +132,8 @@
         </inertial>
     </link> -->
-    <joint name="base_joint" type="fixed">
-        <parent link="base_footprint" />
-        <child link="base_link" />
-        <origin xyz="0 0 ${wheel_radius}" rpy="0 0 0"/>
-    </joint>
     <joint name="base_right_wheel_joint" type="continuous">
         <parent link="base_link" />
         <child link="right_wheel_link" />
-        <origin xyz="0.09 -0.1 0" rpy="0 0 0" />
+        <origin xyz="0.09 -0.09 0" rpy="0 0 0" />
         <axis xyz="0 1 0" />
     </joint>
@@ -141,5 +141,5 @@
         <parent link="base_link" />
         <child link="left_wheel_link" />
-        <origin xyz="0.09 0.1 0" rpy="0 0 0" />
+        <origin xyz="0.09 0.09 0" rpy="0 0 0" />
         <axis xyz="0 1 0" />
     </joint>
@@ -147,5 +147,5 @@
         <parent link="base_link" />
         <child link="rightb_wheel_link" />
-        <origin xyz="-0.09 -0.1 0" rpy="0 0 0" />
+        <origin xyz="-0.09 -0.09 0" rpy="0 0 0" />
         <axis xyz="0 1 0" />
     </joint>
@@ -153,5 +153,5 @@
         <parent link="base_link" />
         <child link="leftb_wheel_link" />
-        <origin xyz="-0.09 0.1 0" rpy="0 0 0" />
+        <origin xyz="-0.09 0.09 0" rpy="0 0 0" />
         <axis xyz="0 1 0" />
     </joint>

File: src/mapper_description/urdf/mobile_base_gazebo.xacro (robot description, xacro)
@@ -54,5 +54,5 @@
         <sensor name="imu_sensor" type="imu">
             <always_on>true</always_on>
-            <update_rate>50</update_rate>
+            <update_rate>20</update_rate>
             <visualize>true</visualize>
             <topic>imu1</topic>

File: src/mapper_description/urdf/sensors.xacro (robot description, xacro)
@@ -1,11 +1,19 @@
 <?xml version="1.0"?>
 <robot xmlns:xacro="http://www.ros.org/wiki/xacro" >
-    <joint name="sonar_front_joint" type="fixed">
+    <!-- Down -->
+    <!-- <joint name="sonar_front_joint" type="fixed">
         <axis xyz="0 1 0" />
-        <origin rpy="0 0 0" xyz="0.16 0 0.09" />
+        <origin rpy="0 0 0" xyz="0 0 0.054" />
         <parent link="base_footprint"/>
         <child link="base_sonar_front"/>
-    </joint>
-    <link name="base_sonar_front">
+    </joint> -->
+    <!-- Front -->
+    <!-- <joint name="sonar_front_joint" type="fixed">
+        <axis xyz="0 1 0" />
+        <origin rpy="0 0.34 0" xyz="0.155 0 0.100" />
+        <parent link="base_link"/>
+        <child link="base_sonar_front"/>
+    </joint> -->
+    <!-- <link name="base_sonar_front">
         <collision>
           <origin xyz="0 0 0" rpy="0 0 0"/>
@@ -26,9 +34,9 @@
           <inertia ixx="1e-6" ixy="0" ixz="0" iyy="1e-6" iyz="0" izz="1e-6" />
         </inertial>
-     </link>
+     </link> -->
     <joint name="lidar_joint" type="fixed">
-        <parent link="base_footprint"/>
+        <parent link="base_link"/>
         <child link="lidar_link"/>
-        <origin xyz="0 0 0.145" rpy="0 0 0"/>
+        <origin xyz="0 0 0.095" rpy="0 0 0"/>
     </joint>
     <link name="lidar_link">
@@ -48,7 +56,7 @@
     </link>
     <joint name="imu_joint" type="fixed">
-        <parent link="base_footprint"/>
+        <parent link="base_link"/>
         <child link="imu_link"/>
-        <origin xyz="0 0 0.09" rpy="0 0 0"/>
+        <origin xyz="0 0 0.04" rpy="0 0 0"/>
     </joint>
     <link name="imu_link">
@@ -56,4 +64,24 @@
             <geometry>
                 <box size="0.05 0.05 0.02"/>
+            </geometry>
+            <material name="grey"/>
+        </visual>
+        <collision>
+            <geometry>
+                <box size="0.1 0.1 0.1"/>
+            </geometry>
+        </collision>
+        <xacro:box_inertia m="0.1" l="0.1" w="0.1" h="0.1"
+                           xyz="0 0 0" rpy="0 0 0" />
+    </link>
+    <joint name="camera_joint" type="fixed">
+        <parent link="base_link"/>
+        <child link="camera_link"/>
+        <origin xyz="0.156 0 0.08" rpy="0 0 0"/>
+    </joint>
+    <link name="camera_link">
+        <visual>
+            <geometry>
+                <box size="0.010 0.06 0.02"/>
             </geometry>
             <material name="grey"/>
@@ -97,7 +125,7 @@
     <gazebo reference="base_sonar_front">
         <sensor type="ray" name="TeraRanger">
-            <pose>0 0 0 0 0 0</pose>
+            <pose>0 0 2 0 0 0</pose>
             <visualize>true</visualize>
-            <update_rate>50</update_rate>
+            <update_rate>20</update_rate>
             <ray>
                 <scan>
@@ -116,19 +144,46 @@
                 </scan>
                 <range>
-                    <min>0.01</min>
-                    <max>2</max>
+                    <min>0.005</min>
+                    <max>5.0</max>
                     <resolution>0.02</resolution>
                 </range>
             </ray>
-            <plugin name="gazebo_ros_range_sensor" filename="libgazebo_ros_ray_sensor.so">
+            <plugin name="sonar_plugin" filename="libgazebo_ros_ray_sensor.so">
                 <ros>
                     <namespace>sensor</namespace>
                     <argument>sonar_front:=sonar_front</argument>
                 </ros>
-                <topicName>/sensor/sonar_front</topicName>
+                <output_type>sensor_msgs/LaserScan</output_type>
+                <topicName>sonar_front</topicName>
                 <frameName>base_sonar_front</frameName>
-                <updateRate>50</updateRate>
-                <gaussianNoise>0.005</gaussianNoise>
-                <radiation>INFRARED</radiation>
+                <updateRate>20</updateRate>
+                <gaussianNoise>0.01</gaussianNoise>
+                <radiation>ultrasound</radiation>
+                <!-- <gaussianNoise>0.005</gaussianNoise>
+                <topicName>sonar</topicName>
+                <frameId>sonar_link</frameId> -->
+            </plugin>
+        </sensor>
+    </gazebo>
+    <gazebo reference="camera_link">
+        <material>Gazebo/Grey</material>
+        <sensor name="camera" type="camera">
+            <pose> 0 0 0 0 0 0 </pose>
+            <visualize>true</visualize>
+            <update_rate>50</update_rate>
+            <camera>
+                <horizontal_fov>1.03</horizontal_fov>
+                <image>
+                    <format>R8G8B8</format>
+                    <width>640</width>
+                    <height>480</height>
+                </image>
+                <clip>
+                    <near>0.05</near>
+                    <far>8.0</far>
+                </clip>
+            </camera>
+            <plugin name="camera_controller" filename="libgazebo_ros_camera.so">
+                <frame_name>camera_link</frame_name>
             </plugin>
         </sensor>
